File: eagle/kelvin_ntc_B.brd (EAGLE design)
At the start: 72 x 42.3 mm, 49 parts, among them IC1 PIC18F2580, IC3 MCP2551SN, IC4 LM2575S, J1 OSTTE-12, J2 A00-108-220-450, Q1 10 MHz

Commit message: added workfiles to ignore list
Connections:
- net N$22 renamed CANH
Routing:
- net CANH: track 43.6 -> 43.0 mm
Changed lines of the file:
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@@
 <via x="43.47" y="29.68" extent="1-16" drill="0.6" shape="square"/>
 </signal>
-<signal name="N$22">
+<signal name="CANH">
 <contactref element="R17" pad="1"/>
 <contactref element="J4" pad="2"/>
@@
 <wire x1="60.12" y1="15.13" x2="59.53" y2="15.72" width="0.254" layer="1"/>
 <wire x1="41.71" y1="11.19" x2="43.34" y2="11.2" width="0.254" layer="1"/>
-<wire x1="43.34" y1="11.2" x2="45.93" y2="11.23" width="0.254" layer="1"/>
-<wire x1="45.93" y1="11.23" x2="45.93" y2="12.93" width="0.254" layer="1"/>
+<wire x1="43.34" y1="11.2" x2="45.13" y2="11.23" width="0.254" layer="1"/>
+<wire x1="45.13" y1="11.23" x2="45.93" y2="12.93" width="0.254" layer="1"/>
 <wire x1="45.93" y1="12.93" x2="45.945" y2="12.945" width="0.254" layer="1"/>
 <wire x1="41.71" y1="8.95" x2="41.71" y2="11.19" width="0.254" layer="1"/>
@@
 <contactref element="PAD1" pad="1"/>
 <wire x1="39.37" y1="8.89" x2="40.64" y2="10.16" width="0.1778" layer="1"/>
-<wire x1="40.64" y1="10.16" x2="43.18" y2="12.7" width="0.1778" layer="16"/>
-<wire x1="43.18" y1="12.7" x2="48.26" y2="12.7" width="0.1778" layer="16"/>
+<wire x1="40.64" y1="10.16" x2="42.98" y2="12.6" width="0.1778" layer="16"/>
+<wire x1="42.98" y1="12.6" x2="48.26" y2="12.7" width="0.1778" layer="16"/>
 <wire x1="48.26" y1="12.7" x2="49.53" y2="13.97" width="0.1778" layer="16"/>
 <wire x1="39.72" y1="8.86" x2="39.37" y2="8.89" width="0.1778" layer="1"/>
